File: project/offzone-addon-s7.kicad_sch (KiCad schematic)
At the start: 14 parts, among them Q1 MMBT3904, U1 TLC555

Commit message: Add EasyEDA version of the schematic
project/offzone-addon-s7-easyeda.json holds the same circuit as the KiCad
sheet, in EasyEDA Standard format (File -> Open -> EasyEDA). Symbols are the
real LCSC ones, so footprints and part numbers come along and the sheet can be
pushed straight to a board.

Nets +3V, GND, TC, DIS, OUT and BLINK are joined by net labels rather than long
wires, which keeps the routing around U1 free of crossings. The netlist is
identical to the KiCad sheet.

Also settle on one timer across both files: LMC555M/TR (C356725, SOP-8), picked
because it is in stock and runs from 1.5 V. The KiCad symbol and value follow.

Co-Authored-By: Claude Opus 5 (1M context) <noreply@anthropic.com>
Parts:
- U1: value TLC555 -> LMC555; symbol Timer:TLC555xx -> Timer:LMC555xx
Changed lines of the file:
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@@
 	)
 	(symbol
-		(lib_id "Timer:TLC555xx")
+		(lib_id "Timer:LMC555xx")
 		(at 63.5 46.99 0)
 		(unit 1)
@@
 		(dnp no)
 		(property "Reference" "U1" (at 55.88 36.83 0) (effects (font (size 1.27 1.27)) (justify left)))
-		(property "Value" "TLC555" (at 67.31 36.83 0) (effects (font (size 1.27 1.27)) (justify left)))
+		(property "Value" "LMC555" (at 67.31 36.83 0) (effects (font (size 1.27 1.27)) (justify left)))
 		(property "Footprint" "" (at 63.5 46.99 0) (effects (font (size 1.27 1.27)) hide))
 		(property "Datasheet" "~" (at 63.5 46.99 0) (effects (font (size 1.27 1.27)) hide))

Commit message: Switch Q1 to KT3153A9 and fix its pin order
The part is KT3153A9 (Dalex / Integral), n-p-n in a KT-46A (SOT-23) package.
Both datasheets agree its pin order is 1 = collector, 2 = base, 3 = emitter,
which is NOT the western SOT-23 order the MMBT3904 symbol used (1 = base,
2 = emitter, 3 = collector). Renaming alone would have wired the transistor
inside out, so the symbol pins are renumbered to match the datasheet.

KiCad now uses Device:Q_NPN_CBE; the EasyEDA sheet renumbers the borrowed
symbol and drops the LCSC part attributes, since this part is sourced locally.

Headroom is ample: 400 mA rating against ~30 mA of load, and h21e 100..300 with
about 2 mA of base current keeps it well into saturation.

Co-Authored-By: Claude Opus 5 (1M context) <noreply@anthropic.com>
Parts:
- Q1: value MMBT3904 -> KT3153A9; symbol Device:Q_NPN_BEC -> Device:Q_NPN_CBE
Connections:
- net BLINK: now also Q1.1 (C); no longer Q1.3 (C)
- net GND: now also Q1.3 (E); no longer Q1.2 (E)
- net at R3.2: now also Q1.2 (B); no longer Q1.1 (B)
Other:
- note added: "Q1 — КТ3153А9 (корпус КТ-46А / SOT-23): вывод 1 — коллектор, 2 — база, 3 — эмиттер (НЕ как у MMBT3904)"
Changed lines of the file:
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@@
+		(effects (font (size 1.27 1.27)) (justify left bottom))
+	)
+	(text "Q1 — КТ3153А9 (корпус КТ-46А / SOT-23): вывод 1 — коллектор, 2 — база, 3 — эмиттер (НЕ как у MMBT3904)" (at 30.48 111.76 0)
 		(effects (font (size 1.27 1.27)) (justify left bottom))
 	)
@@
 	)
 	(symbol
-		(lib_id "Device:Q_NPN_BEC")
+		(lib_id "Device:Q_NPN_CBE")
 		(at 101.6 46.99 0)
 		(unit 1)
@@
 		(dnp no)
 		(property "Reference" "Q1" (at 106.68 48.26 0) (effects (font (size 1.27 1.27)) (justify left)))
-		(property "Value" "MMBT3904" (at 106.68 50.8 0) (effects (font (size 1.27 1.27)) (justify left)))
+		(property "Value" "KT3153A9" (at 106.68 50.8 0) (effects (font (size 1.27 1.27)) (justify left)))
 		(property "Footprint" "" (at 101.6 46.99 0) (effects (font (size 1.27 1.27)) hide))
 		(property "Datasheet" "~" (at 101.6 46.99 0) (effects (font (size 1.27 1.27)) hide))
